File: ISA8019.kicad_pcb (KiCad board)
At the start: 2 copper layers, 53 parts, among them J1 Bus_ISA_16bit, J2 8P8C_Shielded, J3 AUI, J4 Jumper mode, J5 PNP force, J6 BROM size and base address, J7 I/O base address, J8 Medium type, J9 IRQ select, T1 13F-39MNL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

Commit message: Add mechanicals
Parts:
- added H3: MountingHole_Pad, MountingHole:MountingHole_3.2mm_M3_Pad_Via, F.Cu at (188.2, 151.6)
- added H4: MountingHole_Pad, MountingHole:MountingHole_3.2mm_M3_Pad_Via, F.Cu at (188.2, 95.1)
- moved C15 173.5 mm to (-38.9, 28.3)
- moved C4 173.5 mm to (-20.1, 11.4)
- moved C5 173.5 mm to (-34.5, 26.3)
- moved C6 173.5 mm to (-34.5, 24.3)
- moved J3 173.5 mm to (-53.8, 8.73)
- moved J5 173.5 mm to (-39.4, 21.0)
- moved J7 173.5 mm to (-39.4, 8.73)
- moved R10 173.5 mm to (-23.0, 9.39)
- moved R11 173.5 mm to (-23.0, 13.4)
- moved R12 173.5 mm to (-25.9, 11.4)
- moved R15 173.5 mm to (-25.9, 15.4)
- moved R17 173.5 mm to (-25.9, 13.4)
- moved R18 173.5 mm to (-23.0, 11.4)
- moved R19 173.5 mm to (-41.8, 28.3)
- moved R22 173.5 mm to (-25.9, 7.40)
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Routing:
- added copper zone on B.Cu, net GND
- added copper zone on F.Cu, net GND
Other:
- board outline added: 157.4 x 74.2 mm
- net class Default: clearance 0.2 -> 0.127; trace_width 0.25 -> 0.127; via_dia 0.8 -> 0.6; via_drill 0.4 -> 0.3
- rule trace_clearance: 0.2 -> 0.127
- rule trace_min: 0.2 -> 0.127
- rule via_min_size: 0.4 -> 0.6

Commit message: Some routing
Parts:
- removed J3: AUI, Connector_PinHeader_2.54mm:PinHeader_2x08_P2.54mm_Vertical
- added FB1: Ferrite_Bead, Inductor_SMD:L_0805_2012Metric, F.Cu at (180.7, 125.9)
- moved C2 257.7 mm to (188.0, 135.3)
- moved R8 222.2 mm to (175.5, 79.4), turned to 90 degrees
- moved J4 221.8 mm to (169.2, 74.9), turned to 90 degrees
- moved J5 221.6 mm to (175.5, 74.9), turned to 90 degrees
- moved R19 210.9 mm to (162.8, 79.4), turned to 90 degrees
- moved R7 207.2 mm to (169.2, 79.4), turned to 90 degrees
- moved J8 200.6 mm to (160.3, 74.9), turned to 90 degrees
- moved R18 195.4 mm to (160.3, 79.4), turned to 90 degrees
- moved R21 195.4 mm to (150.1, 79.4), turned to 90 degrees
- moved C15 194.5 mm to (126.4, 130.8)
- moved R22 192.5 mm to (152.7, 79.4), turned to 90 degrees
- moved R20 192.4 mm to (147.6, 79.4), turned to 90 degrees
- moved J9 191.6 mm to (147.6, 74.9), turned to 90 degrees
- moved C3 189.3 mm to (112.1, 146.8), turned to 270 degrees
- moved C4 183.4 mm to (103.9, 146.6), turned to 225 degrees
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Connections:
- J6 pad 2: Net-(J6-Pad2) -> +5V
- J6 pad 4: Net-(J6-Pad4) -> +5V
- J6 pad 7: +5V -> Net-(J6-Pad7)
- J6 pad 9: +5V -> Net-(J6-Pad9)
- J7 pad 2: Net-(J7-Pad2) -> +5V
- J7 pad 4: Net-(J7-Pad4) -> +5V
- J7 pad 5: +5V -> Net-(J7-Pad5)
- J7 pad 7: +5V -> Net-(J7-Pad7)
- J8 pad 2: Net-(J8-Pad2) -> +5V
- J8 pad 3: +5V -> Net-(J8-Pad3)
- J9 pad 2: Net-(J9-Pad2) -> +5V
- J9 pad 5: +5V -> Net-(J9-Pad5)
- R10 pad 2: Net-(J6-Pad2) -> Net-(J6-Pad7)
- R11 pad 2: Net-(J6-Pad3) -> Net-(J6-Pad5)
- R12 pad 2: Net-(J6-Pad4) -> Net-(J6-Pad3)
- R13 pad 2: Net-(J6-Pad5) -> Net-(J6-Pad1)
- R15 pad 2: Net-(J7-Pad2) -> Net-(J7-Pad3)
- R16 pad 2: Net-(J7-Pad3) -> Net-(J7-Pad5)
- R17 pad 2: Net-(J7-Pad4) -> Net-(J7-Pad7)
- R19 pad 2: Net-(J8-Pad2) -> Net-(J8-Pad3)
- R21 pad 2: Net-(J9-Pad2) -> Net-(J9-Pad3)
- R22 pad 2: Net-(J9-Pad3) -> Net-(J9-Pad5)
- R9 pad 2: Net-(J6-Pad1) -> Net-(J6-Pad9)
- Y1 pad 1: Net-(C8-Pad2) -> Net-(C9-Pad2)
- Y1 pad 3: Net-(C9-Pad2) -> Net-(C8-Pad2)
Routing:
- net /ISA_D15: track 0.00 -> 88.5 mm, vias 0 -> 2
- net /ISA_D14: track 0.00 -> 84.5 mm, vias 0 -> 2
- net /ISA_D13: track 0.00 -> 80.7 mm, vias 0 -> 2
- net /ISA_D12: track 0.00 -> 77.2 mm, vias 0 -> 2
- net /ISA_D11: track 0.00 -> 74.5 mm, vias 0 -> 2
- net /ISA_D10: track 0.00 -> 70.0 mm, vias 0 -> 2
- net /ISA_D9: track 0.00 -> 66.4 mm, vias 0 -> 2
- net /ISA_D8: track 0.00 -> 62.9 mm, vias 0 -> 2
- net /ISA_D7: track 0.00 -> 61.0 mm
- net /ISA_RESET: track 0.00 -> 60.5 mm, vias 0 -> 1
- net /ISA_D6: track 0.00 -> 58.4 mm
- net /ISA_D5: track 0.00 -> 55.7 mm
- net /TPIN+: track 0.00 -> 54.3 mm, vias 0 -> 2
- net /TPIN-: track 0.00 -> 53.5 mm, vias 0 -> 2
- net /ISA_D4: track 0.00 -> 52.7 mm
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- added copper zone on F.Cu, net Earth

Commit message: some routing later
Parts:
- J4: value Jumper mode -> JP
- moved U3 43.9 mm to (42.7, 110.0), turned to 90 degrees
- moved J4 15.5 mm to (153.7, 73.7)
- moved J5 15.5 mm to (160.0, 73.7)
- moved J8 15.5 mm to (144.8, 73.7)
- moved J9 15.5 mm to (132.1, 73.7)
- moved R18 15.5 mm to (144.8, 78.1)
- moved R19 15.5 mm to (147.3, 78.1)
- moved R20 15.5 mm to (132.1, 78.1)
- moved R21 15.5 mm to (134.6, 78.1)
- moved R22 15.5 mm to (137.2, 78.1)
- moved R7 15.5 mm to (153.7, 78.1)
- moved R8 15.5 mm to (160.0, 78.1)
- moved C3 10.2 mm to (112.1, 136.7)
- moved C6 10.2 mm to (95.2, 123.9)
- moved C9 10.2 mm to (123.4, 113.4)
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Routing:
- net /ISA_D7: track 61.0 -> 0.00 mm
- net /ISA_RESET: track 60.5 -> 1.76 mm
- net /ISA_D6: track 58.4 -> 0.00 mm
- net /ISA_D5: track 55.7 -> 0.00 mm
- net /ISA_D4: track 52.7 -> 0.00 mm
- net /ISA_D3: track 50.2 -> 0.00 mm
- net /ISA_A0: track 22.0 -> 72.1 mm, vias 0 -> 1
- net /ISA_D2: track 47.3 -> 0.00 mm
- net /ISA_D1: track 44.8 -> 0.00 mm
- net /ISA_D0: track 42.4 -> 0.00 mm
- net /~ISA_IOW: track 0.00 -> 41.6 mm, vias 0 -> 3
- net /ISA_IO_CH_RDY: track 39.5 -> 0.00 mm
- net /TPOUT+: track 46.8 -> 7.77 mm
- net /TPOUT-: track 46.9 -> 7.85 mm
- net /ISA_AEN: track 36.6 -> 0.00 mm
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
Commit message: Redo most of the bus layout
Parts:
- moved U2 30.4 mm to (71.8, 109.8), turned to 270 degrees
- moved J4 25.7 mm to (149.9, 99.1)
- moved J5 25.7 mm to (156.2, 99.1)
- moved J6 25.7 mm to (108.0, 99.1)
- moved J7 25.7 mm to (90.2, 99.1)
- moved J8 25.7 mm to (141.0, 99.1)
- moved J9 25.7 mm to (128.3, 99.1)
- moved R12 25.7 mm to (110.5, 103.0)
- moved R13 25.7 mm to (108.0, 103.0)
- moved R15 25.7 mm to (92.7, 102.9)
- moved R10 25.7 mm to (115.6, 103.1)
- moved R11 25.7 mm to (113.0, 103.1)
- moved R14 25.7 mm to (90.2, 102.7)
- moved R16 25.7 mm to (95.2, 102.7)
- moved R17 25.7 mm to (97.8, 102.7)
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Routing:
- net /ISA_A13: track 7.16 -> 122.3 mm
- net /ISA_A8: track 10.4 -> 113.8 mm
- net /BA14: track 0.00 -> 102.5 mm
- net /ISA_A12: track 7.81 -> 108.7 mm
- net /ISA_A9: track 9.76 -> 110.6 mm
- net /ISA_A11: track 8.46 -> 108.3 mm
- net /BA15: track 0.00 -> 99.2 mm
- net /ISA_A10: track 9.11 -> 102.7 mm
- net /ISA_A6: track 11.1 -> 98.9 mm
- net /BA16: track 0.00 -> 85.2 mm
- net /ISA_A5: track 11.7 -> 96.0 mm
- net /ISA_A4: track 12.4 -> 93.0 mm
- net /ISA_A3: track 13.0 -> 91.1 mm
- net /ISA_A7: track 25.5 -> 101.8 mm, vias 0 -> 1
- net /ISA_A2: track 14.5 -> 88.7 mm
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